Commit message: fix: urdf joint frictions and dampings

File: urdfs/d1h_description/xacro/d1h_base.xacro (robot description, xacro)
@@ -130,5 +130,5 @@
       <child link="${name}L_hip"/>
       <axis xyz="1 0 0" />
-      <dynamics damping="0.2346" friction="0.943"/>
+      <dynamics damping="0.05" friction="0.15"/>
       <limit lower="-0.7854" upper="0.7854" effort="80" velocity="20" />
     </joint>
@@ -162,5 +162,5 @@
       <child link="${name}L_thigh" />
       <axis xyz="0 1 0" />
-      <dynamics damping="0.2346" friction="0.943"/>
+      <dynamics damping="0.05" friction="0.15"/>
       <limit lower="-1.8326" upper="3.4034" effort="80" velocity="20" />
     </joint>
@@ -194,5 +194,5 @@
       <child link="${name}L_calf" />
       <axis xyz="0 1 0" />
-      <dynamics damping="0.2346" friction="0.943"/>
+      <dynamics damping="0.05" friction="0.15"/>
       <limit lower="-2.72" upper="-0.85" effort="80" velocity="20" />
     </joint>
@@ -226,5 +226,5 @@
       <child link="${name}L_foot" />
       <axis xyz="0 1 0" />
-      <dynamics damping="0.5" friction="0.0"/>
+      <dynamics damping="0.005" friction="0.02"/>
       <limit lower="-31415926" upper="31415926" effort="12" velocity="30" />
     </joint>
@@ -252,5 +252,5 @@
       <child link="${name}R_hip" />
       <axis xyz="1 0 0" />
-      <dynamics damping="0.2346" friction="0.943"/>
+      <dynamics damping="0.05" friction="0.15"/>
       <limit lower="-0.7854" upper="0.7854" effort="80" velocity="20" />
     </joint>
@@ -284,5 +284,5 @@
       <child link="${name}R_thigh" />
       <axis xyz="0 1 0" />
-      <dynamics damping="0.2346" friction="0.943"/>
+      <dynamics damping="0.05" friction="0.15"/>
       <limit lower="-1.8326" upper="3.4034" effort="80" velocity="20" />
     </joint>
@@ -316,5 +316,5 @@
       <child link="${name}R_calf" />
       <axis xyz="0 1 0" />
-      <dynamics damping="0.2346" friction="0.943"/>
+      <dynamics damping="0.05" friction="0.15"/>
       <limit lower="-2.72" upper="-0.85" effort="80" velocity="20" />
     </joint>
@@ -348,5 +348,5 @@
       <child link="${name}R_foot" />
       <axis xyz="0 1 0" />
-      <dynamics damping="0.5" friction="0.0"/>
+      <dynamics damping="0.005" friction="0.02"/>
       <limit lower="-31415926" upper="31415926" effort="12" velocity="30" />
     </joint>
